Commit message: Changed pantograph description to account for new world frame definition

File: pantograph_description/urdf/pantograph.urdf.xacro (robot description, xacro)
@@ -21,5 +21,5 @@
       </geometry>
       <material name = "white_alpha"/>
-      <origin xyz="0 0 0" rpy="0 0 0" />
+      <origin xyz="-0.0425 0 0" rpy="0 0 0" />
     </visual>
   </link>
@@ -42,5 +42,5 @@
     <parent link = "panto_base"/>
     <child link = "panto_link_fulcrum"/>
-    <origin xyz = "0.0425 0.16056 0.09"/>
+    <origin xyz = "0.0 0.16056 0.09"/>
   </joint>
   <!-- ==========  Left arm (as seen from behind) =========== -->
@@ -55,5 +55,5 @@
     <parent link = "panto_base"/>
     <child link = "panto_left_motor"/>
-    <origin xyz = "0.0 0 0" rpy="0 0 0"/>
+    <origin xyz = "-0.0425 0 0" rpy="0 0 0"/>
     <limit effort="1000.0" lower="-1.57" upper="1.57" velocity="0.5"/>
     <axis xyz = "0 0 1"/>
@@ -120,5 +120,5 @@
     <parent link = "panto_base"/>
     <child link = "panto_right_motor"/>
-    <origin xyz = "0.085 0 0" rpy="0 0 0"/>
+    <origin xyz = "0.0425 0 0" rpy="0 0 0"/>
     <limit effort="1000.0" lower="-1.57" upper="1.57" velocity="0.5"/>
     <axis xyz = "0 0 1"/>
@@ -160,5 +160,6 @@
   <link name="tool_theta_link"/>
   <joint name="tool_theta_joint" type="continuous">
-    <parent link= "panto_tool0"/>
+    <!-- <parent link= "panto_tool0"/> -->
+    <parent link= "panto_link_fulcrum"/>
     <child link= "tool_theta_link"/>
     <origin xyz = "0 0 0" rpy="0 0 0"/>
@@ -169,8 +170,8 @@
     <visual>
       <geometry>
-        <cylinder length = "0.2" radius = "0.0025"/>
+        <cylinder length = "0.15" radius = "0.0025"/>
       </geometry>
       <material name = "white_alpha"/>
-      <origin xyz = "0 0 0.1" rpy = "0 0 0"/>
+      <origin xyz = "0 0 -0.075" rpy = "0 0 0"/>
     </visual>
   </link>

Commit message: Update robot description and models

File: pantograph_description/urdf/pantograph.urdf.xacro (robot description, xacro)
@@ -187,5 +187,5 @@
     <parent link= "tool_phi_link"/>
     <child link= "needle_interaction_link"/>
-    <origin xyz = "0 0 0.1" rpy="0 0 0"/>
+    <origin xyz = "0 0 0.05" rpy="0 0 0"/>
     <limit effort="1000.0" lower="0.5" upper="-0.5" velocity="0.5"/>
     <axis xyz="0 0 1"/>
